File: Arduino_USB_C/arduino_usb_c/arduino_usb_c.kicad_sch (KiCad schematic)
At the start: 47 parts, among them J1 USB_C_Receptacle_USB2.0, J2 Conn_02x03_Odd_Even, J3 Screw_Terminal_01x02, J4 Screw_Terminal_01x02, J5 Conn_01x03_Male, J6 Conn_02x03_Odd_Even, J7 Conn_01x03_Male, J8 Conn_01x03_Male, SW1 SW_SPST, SW2 SW_SPST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

Commit message: added step files
Parts:
- J1: Digikey (none) -> 2073-USB4105-GF-ACT-ND
- J2: Digikey https://www.digikey.com/en/products/detail/harwin-inc/M20-9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 -> 952-2121-ND
- J3, J4: Digikey (none) -> 796949-2-ND
- SW1: Digikey (none) -> CKN12326-1-ND
- U4: Digikey (none) -> 785-1670-1-ND
Changed lines of the file:
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@@
+      (effects (font (size 1.27 1.27)) hide)
+    )
+    (property "Digikey" "796949-2-ND" (id 4) (at 152.4 133.985 0)
       (effects (font (size 1.27 1.27)) hide)
     )
@@
       (effects (font (size 1.27 1.27)) hide)
     )
+    (property "Digikey" "CKN12326-1-ND" (id 4) (at 71.12 36.83 0)
+      (effects (font (size 1.27 1.27)) hide)
+    )
     (pin "1")
     (pin "2")
@@
     )
     (property "Datasheet" "https://www.usb.org/sites/default/files/documents/usb_type-c.zip" (id 3) (at 144.78 45.085 0)
+      (effects (font (size 1.27 1.27)) hide)
+    )
+    (property "Digikey" "2073-USB4105-GF-ACT-ND" (id 4) (at 140.97 45.085 0)
       (effects (font (size 1.27 1.27)) hide)
     )
@@
     )
     (property "Datasheet" "~" (id 3) (at 142.24 158.75 0)
+      (effects (font (size 1.27 1.27)) hide)
+    )
+    (property "Digikey" "796949-2-ND" (id 4) (at 142.24 158.75 0)
       (effects (font (size 1.27 1.27)) hide)
     )
@@
       (effects (font (size 1.27 1.27)) hide)
     )
+    (property "Digikey" "785-1670-1-ND" (id 4) (at 176.53 133.985 0)
+      (effects (font (size 1.27 1.27)) hide)
+    )
     (pin "1")
     (pin "2")
@@
       (effects (font (size 1.27 1.27)) hide)
     )
-    (property "Datasheet" "~" (id 3) (at 172.72 76.835 0)
-      (effects (font (size 1.27 1.27)) hide)
-    )
-    (property "Digikey" "https://www.digikey.com/en/products/detail/harwin-inc/M20-9980346/3728085" (id 4) (at 172.72 76.835 0)
-      (effects (font (size 1.27 1.27)) hide)
-    )
+    (property "Datasheet" "https://www.digikey.com/en/products/detail/harwin-inc/M20-9980346/3728085" (id 3) (at 172.72 76.835 0)
+      (effects (font (size 1.27 1.27)) hide)
+    )
+    (property "Digikey" "952-2121-ND" (id 4) (at 172.72 76.835 0)
+      (effects (font (size 1.27 1.27)) hide)
+    )
